Commit message: update collision mesh

File: robot_description/rccn_kuka_robot_cell/urdf/rccn_east_robot.xacro (robot description, xacro)
@@ -12,5 +12,5 @@
             <collision>
                 <geometry>
-                    <mesh filename="package://rccn_kuka_robot_cell/meshes/world/collision/robot_cell_fixture.stl"/>
+                    <mesh scale="0.001 0.001 0.001" filename="package://rccn_kuka_robot_cell/meshes/world/collision/robot_cell_fixture.stl"/>
                 </geometry>
             </collision>

File: robot_description/rccn_kuka_robot_cell/urdf/rccn_east_robot_macro.xacro (robot description, xacro)
@@ -15,5 +15,5 @@
                 <collision>
                     <geometry>
-                        <mesh filename="package://rccn_kuka_robot_cell/meshes/rail/collision/east_rail.stl"/>
+                        <mesh scale="0.001 0.001 0.001" filename="package://rccn_kuka_robot_cell/meshes/rail/collision/east_rail.stl"/>
                     </geometry>
                 </collision>
@@ -40,5 +40,5 @@
                 <collision>
                     <geometry>
-                        <mesh filename="package://rccn_kuka_robot_cell/meshes/rail/collision/east_plate.stl"/>
+                        <mesh scale="0.001 0.001 0.001" filename="package://rccn_kuka_robot_cell/meshes/rail/collision/east_plate.stl"/>
                     </geometry>
                 </collision>

File: robot_description/rccn_kuka_robot_cell/urdf/rccn_kuka_robot_cell.xacro (robot description, xacro)
@@ -12,5 +12,5 @@
             <collision>
                 <geometry>
-                    <mesh filename="package://rccn_kuka_robot_cell/meshes/world/collision/robot_cell_fixture.stl"/>
+                    <mesh scale="0.001 0.001 0.001" filename="package://rccn_kuka_robot_cell/meshes/world/collision/robot_cell_fixture.stl"/>
                 </geometry>
             </collision>

File: robot_description/rccn_kuka_robot_cell/urdf/rccn_west_robot.xacro (robot description, xacro)
@@ -12,5 +12,5 @@
             <collision>
                 <geometry>
-                    <mesh filename="package://rccn_kuka_robot_cell/meshes/world/collision/robot_cell_fixture.stl"/>
+                    <mesh scale="0.001 0.001 0.001" filename="package://rccn_kuka_robot_cell/meshes/world/collision/robot_cell_fixture.stl"/>
                 </geometry>
             </collision>

File: robot_description/rccn_kuka_robot_cell/urdf/rccn_west_robot_macro.xacro (robot description, xacro)
@@ -15,5 +15,5 @@
                 <collision>
                     <geometry>
-                        <mesh filename="package://rccn_kuka_robot_cell/meshes/rail/collision/west_rail.stl"/>
+                        <mesh scale="0.001 0.001 0.001" filename="package://rccn_kuka_robot_cell/meshes/rail/collision/west_rail.stl"/>
                     </geometry>
                 </collision>
@@ -40,5 +40,5 @@
                 <collision>
                     <geometry>
-                        <mesh filename="package://rccn_kuka_robot_cell/meshes/rail/collision/west_plate.stl"/>
+                        <mesh scale="0.001 0.001 0.001" filename="package://rccn_kuka_robot_cell/meshes/rail/collision/west_plate.stl"/>
                     </geometry>
                 </collision>
