Commit message: update urdf to use binary urdf

File: robot_description/rccn_kuka_robot_cell/urdf/rccn_west_robot.urdf (robot description, URDF)
Before this commit: robot rccn_west_robot, 12 links, 11 joints
Links:
- link kuka_robot_cell_world: geometry collision mesh filename=package://rccn_kuka_robot_cell/meshes/world/collision/robot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 scale=0.001 0.001 0.001; visual mesh filename=package://rccn_kuka_robot_cell/meshes/world/visual/robot_ce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
- link west_e1_plate: geometry collision mesh filename=package://rccn_kuka_robot_cell/meshes/rail/collision/west_p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 scale=0.001 0.001 0.001; visual mesh filename=package://rccn_kuka_robot_cell/meshes/rail/visual/west_plat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
- link west_e1_rail: geometry collision mesh filename=package://rccn_kuka_robot_cell/meshes/rail/collision/west_r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 scale=0.001 0.001 0.001; visual mesh filename=package://rccn_kuka_robot_cell/meshes/rail/visual/west_rail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

Commit message: use simple floor mesh

File: robot_description/rccn_kuka_robot_cell/urdf/rccn_west_robot.urdf (robot description, URDF)
Before this commit: robot rccn_west_robot, 12 links, 11 joints
Links:
- link kuka_robot_cell_world: geometry collision mesh filename=package://rccn_kuka_robot_cell/meshes/world/collision/floor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 scale=0.001 0.001 0.001; visual mesh filename=package://rccn_kuka_robot_cell/meshes/world/visual/robot_ce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

File: robot_description/rccn_kuka_robot_cell/urdf/rccn_west_robot.xacro (robot description, xacro)
@@ -12,5 +12,5 @@
             <collision>
                 <geometry>
-                    <mesh scale="0.001 0.001 0.001" filename="package://rccn_kuka_robot_cell/meshes/world/collision/robot_cell_fixture.stl"/>
+                    <mesh scale="0.001 0.001 0.001" filename="package://rccn_kuka_robot_cell/meshes/world/collision/floor.stl"/>
                 </geometry>
             </collision>
