Commit message: Update URDF files and moveit configuration for KUKA KR300 R2500 ultra

File: robot_description/rccn_kuka_robot_cell/urdf/rccn_east_robot.urdf (robot description, URDF)
Before this commit: robot rccn_east_robot, 11 links, 10 joints
Links:
- added link east_base
- link east_base_link: geometry collision mesh filename=package://kuka_kr300_support/meshes/kr300r2500ultra/collisi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 scale=0.001 0.001 0.001; visual mesh filename=package://kuka_kr300_support/meshes/kr300r2500ultra/visual/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
- link east_link_1: geometry collision mesh filename=package://kuka_kr300_support/meshes/kr300r2500ultra/collisi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 scale=0.001 0.001 0.001; visual mesh filename=package://kuka_kr300_support/meshes/kr300r2500ultra/visual/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
- link east_link_2: geometry collision mesh filename=package://kuka_kr300_support/meshes/kr300r2500ultra/collisi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 scale=0.001 0.001 0.001; visual mesh filename=package://kuka_kr300_support/meshes/kr300r2500ultra/visual/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
- link east_link_3: geometry collision mesh filename=package://kuka_kr300_support/meshes/kr300r2500ultra/collisi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 scale=0.001 0.001 0.001; visual mesh filename=package://kuka_kr300_support/meshes/kr300r2500ultra/visual/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
- link east_link_4: geometry collision mesh filename=package://kuka_kr300_support/meshes/kr300r2500ultra/collisi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 scale=0.001 0.001 0.001; visual mesh filename=package://kuka_kr300_support/meshes/kr300r2500ultra/visual/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
- link east_link_5: geometry collision mesh filename=package://kuka_kr300_support/meshes/kr300r2500ultra/collisi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 scale=0.001 0.001 0.001; visual mesh filename=package://kuka_kr300_support/meshes/kr300r2500ultra/visual/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
- link east_link_6: geometry collision mesh filename=package://kuka_kr300_support/meshes/kr300r2500ultra/collisi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 scale=0.001 0.001 0.001; visual mesh filename=package://kuka_kr300_support/meshes/kr300r2500ultra/visual/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
Joints:
- added joint east_base_link-base: type fixed, parent east_base_link, child east_base, origin xyz=0 0 0 rpy=0 0 0

File: robot_description/rccn_kuka_robot_cell/urdf/rccn_east_robot_macro.xacro (robot description, xacro)
@@ -3,5 +3,5 @@
         <xacro:macro name="rccn_east_robot" params="prefix">
             <xacro:property name="east_prefix" value="east_" />
-            <xacro:include filename="$(find kuka_kr300_support)/urdf/kr300r2500pro_macro.xacro" />
+            <xacro:include filename="$(find kuka_kr300_support)/urdf/kr300r2500ultra_macro.xacro" />
             <link name="${prefix}east_e1_rail">
                 <visual>
@@ -49,6 +49,6 @@
                 <origin xyz="-0.00206000 -0.00032000 -0.00000000" rpy="-0.00000002 -0.00012841 0.00024798" />
             </joint>
-            <!-- kuka kr300 r2500 pro -->
-            <xacro:kuka_kr300r2500pro prefix="${east_prefix}"/>
+            <!-- kuka kr 300 r2500 ultra -->
+            <xacro:kuka_kr300r2500ultra prefix="${east_prefix}"/>
         </xacro:macro>
     </robot>

File: robot_description/rccn_kuka_robot_cell/urdf/rccn_kuka_robot_cell.urdf (robot description, URDF)
Before this commit: robot rccn_kuka_robot_cell, 21 links, 20 joints
Links:
- added link east_base
- added link west_base
- link east_base_link: geometry collision mesh filename=package://kuka_kr300_support/meshes/kr300r2500ultra/collisi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 scale=0.001 0.001 0.001; visual mesh filename=package://kuka_kr300_support/meshes/kr300r2500ultra/visual/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
- link east_link_1: geometry collision mesh filename=package://kuka_kr300_support/meshes/kr300r2500ultra/collisi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 scale=0.001 0.001 0.001; visual mesh filename=package://kuka_kr300_support/meshes/kr300r2500ultra/visual/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
- link east_link_2: geometry collision mesh filename=package://kuka_kr300_support/meshes/kr300r2500ultra/collisi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 scale=0.001 0.001 0.001; visual mesh filename=package://kuka_kr300_support/meshes/kr300r2500ultra/visual/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
- link east_link_3: geometry collision mesh filename=package://kuka_kr300_support/meshes/kr300r2500ultra/collisi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 scale=0.001 0.001 0.001; visual mesh filename=package://kuka_kr300_support/meshes/kr300r2500ultra/visual/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
- link east_link_4: geometry collision mesh filename=package://kuka_kr300_support/meshes/kr300r2500ultra/collisi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 scale=0.001 0.001 0.001; visual mesh filename=package://kuka_kr300_support/meshes/kr300r2500ultra/visual/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
- link east_link_5: geometry collision mesh filename=package://kuka_kr300_support/meshes/kr300r2500ultra/collisi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 scale=0.001 0.001 0.001; visual mesh filename=package://kuka_kr300_support/meshes/kr300r2500ultra/visual/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
- link east_link_6: geometry collision mesh filename=package://kuka_kr300_support/meshes/kr300r2500ultra/collisi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 scale=0.001 0.001 0.001; visual mesh filename=package://kuka_kr300_support/meshes/kr300r2500ultra/visual/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
- link west_base_link: geometry collision mesh filename=package://kuka_kr300_support/meshes/kr300r2500ultra/collisi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 scale=0.001 0.001 0.001; visual mesh filename=package://kuka_kr300_support/meshes/kr300r2500ultra/visual/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
- link west_link_1: geometry collision mesh filename=package://kuka_kr300_support/meshes/kr300r2500ultra/collisi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 scale=0.001 0.001 0.001; visual mesh filename=package://kuka_kr300_support/meshes/kr300r2500ultra/visual/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
- link west_link_2: geometry collision mesh filename=package://kuka_kr300_support/meshes/kr300r2500ultra/collisi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 scale=0.001 0.001 0.001; visual mesh filename=package://kuka_kr300_support/meshes/kr300r2500ultra/visual/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
- link west_link_3: geometry collision mesh filename=package://kuka_kr300_support/meshes/kr300r2500ultra/collisi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 scale=0.001 0.001 0.001; visual mesh filename=package://kuka_kr300_support/meshes/kr300r2500ultra/visual/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
- link west_link_4: geometry collision mesh filename=package://kuka_kr300_support/meshes/kr300r2500ultra/collisi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 scale=0.001 0.001 0.001; visual mesh filename=package://kuka_kr300_support/meshes/kr300r2500ultra/visual/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
- link west_link_5: geometry collision mesh filename=package://kuka_kr300_support/meshes/kr300r2500ultra/collisi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 scale=0.001 0.001 0.001; visual mesh filename=package://kuka_kr300_support/meshes/kr300r2500ultra/visual/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
- link west_link_6: geometry collision mesh filename=package://kuka_kr300_support/meshes/kr300r2500ultra/collisi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 scale=0.001 0.001 0.001; visual mesh filename=package://kuka_kr300_support/meshes/kr300r2500ultra/visual/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
Joints:
- added joint east_base_link-base: type fixed, parent east_base_link, child east_base, origin xyz=0 0 0 rpy=0 0 0
- added joint west_base_link-base: type fixed, parent west_base_link, child west_base, origin xyz=0 0 0 rpy=0 0 0

File: robot_description/rccn_kuka_robot_cell/urdf/rccn_west_robot.urdf (robot description, URDF)
Before this commit: robot rccn_west_robot, 11 links, 10 joints
Links:
- added link west_base
- link west_base_link: geometry collision mesh filename=package://kuka_kr300_support/meshes/kr300r2500ultra/collisi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 scale=0.001 0.001 0.001; visual mesh filename=package://kuka_kr300_support/meshes/kr300r2500ultra/visual/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
- link west_link_1: geometry collision mesh filename=package://kuka_kr300_support/meshes/kr300r2500ultra/collisi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 scale=0.001 0.001 0.001; visual mesh filename=package://kuka_kr300_support/meshes/kr300r2500ultra/visual/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
- link west_link_2: geometry collision mesh filename=package://kuka_kr300_support/meshes/kr300r2500ultra/collisi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 scale=0.001 0.001 0.001; visual mesh filename=package://kuka_kr300_support/meshes/kr300r2500ultra/visual/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
- link west_link_3: geometry collision mesh filename=package://kuka_kr300_support/meshes/kr300r2500ultra/collisi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 scale=0.001 0.001 0.001; visual mesh filename=package://kuka_kr300_support/meshes/kr300r2500ultra/visual/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
- link west_link_4: geometry collision mesh filename=package://kuka_kr300_support/meshes/kr300r2500ultra/collisi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 scale=0.001 0.001 0.001; visual mesh filename=package://kuka_kr300_support/meshes/kr300r2500ultra/visual/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
- link west_link_5: geometry collision mesh filename=package://kuka_kr300_support/meshes/kr300r2500ultra/collisi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 scale=0.001 0.001 0.001; visual mesh filename=package://kuka_kr300_support/meshes/kr300r2500ultra/visual/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
- link west_link_6: geometry collision mesh filename=package://kuka_kr300_support/meshes/kr300r2500ultra/collisi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 scale=0.001 0.001 0.001; visual mesh filename=package://kuka_kr300_support/meshes/kr300r2500ultra/visual/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
Joints:
- added joint west_base_link-base: type fixed, parent west_base_link, child west_base, origin xyz=0 0 0 rpy=0 0 0

File: robot_description/rccn_kuka_robot_cell/urdf/rccn_west_robot_macro.xacro (robot description, xacro)
@@ -3,5 +3,5 @@
         <xacro:macro name="rccn_west_robot" params="prefix">
             <xacro:property name="west_prefix" value="west_" />
-            <xacro:include filename="$(find kuka_kr300_support)/urdf/kr300r2500pro_macro.xacro" />
+            <xacro:include filename="$(find kuka_kr300_support)/urdf/kr300r2500ultra_macro.xacro" />
             <link name="${prefix}west_e1_rail">
                 <visual>
@@ -49,6 +49,6 @@
                 <origin xyz="-0.00043000 -0.00044000 -0.00000000" rpy="0.00000184 0.00009015 0.00206101" />
             </joint>
-            <!-- kuka kr300 r2500 pro -->
-            <xacro:kuka_kr300r2500pro prefix="${west_prefix}"/>
+            <!-- kuka kr 300 r2500 ultra -->
+            <xacro:kuka_kr300r2500ultra prefix="${west_prefix}"/>
         </xacro:macro>
     </robot>

Commit message: modify world collision mesh

File: robot_description/rccn_kuka_robot_cell/urdf/rccn_east_robot.urdf (robot description, URDF)
Before this commit: robot rccn_east_robot, 12 links, 11 joints
Links:
- link east_e1_plate: geometry collision mesh filename=package://rccn_kuka_robot_cell/meshes/rail/collision/east_p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 scale=0.001 0.001 0.001; visual mesh filename=package://rccn_kuka_robot_cell/meshes/rail/visual/east_plat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
- link east_e1_rail: geometry collision mesh filename=package://rccn_kuka_robot_cell/meshes/rail/collision/east_r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 scale=0.001 0.001 0.001; visual mesh filename=package://rccn_kuka_robot_cell/meshes/rail/visual/east_rail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
- link kuka_robot_cell_world: geometry collision mesh filename=package://rccn_kuka_robot_cell/meshes/world/collision/floor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 scale=0.001 0.001 0.001; visual mesh filename=package://rccn_kuka_robot_cell/meshes/world/visual/robot_ce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

File: robot_description/rccn_kuka_robot_cell/urdf/rccn_east_robot.xacro (robot description, xacro)
@@ -12,5 +12,5 @@
             <collision>
                 <geometry>
-                    <mesh scale="0.001 0.001 0.001" filename="package://rccn_kuka_robot_cell/meshes/world/collision/robot_cell_fixture.stl"/>
+                    <mesh scale="0.001 0.001 0.001" filename="package://rccn_kuka_robot_cell/meshes/world/collision/floor.stl"/>
                 </geometry>
             </collision>

File: robot_description/rccn_kuka_robot_cell/urdf/rccn_kuka_robot_cell.urdf (robot description, URDF)
Before this commit: robot rccn_kuka_robot_cell, 23 links, 22 joints
Links:
- link east_e1_plate: geometry collision mesh filename=package://rccn_kuka_robot_cell/meshes/rail/collision/east_p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 scale=0.001 0.001 0.001; visual mesh filename=package://rccn_kuka_robot_cell/meshes/rail/visual/east_plat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
- link east_e1_rail: geometry collision mesh filename=package://rccn_kuka_robot_cell/meshes/rail/collision/east_r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 scale=0.001 0.001 0.001; visual mesh filename=package://rccn_kuka_robot_cell/meshes/rail/visual/east_rail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
- link kuka_robot_cell_world: geometry collision mesh filename=package://rccn_kuka_robot_cell/meshes/world/collision/floor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 scale=0.001 0.001 0.001; visual mesh filename=package://rccn_kuka_robot_cell/meshes/world/visual/robot_ce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
- link west_e1_plate: geometry collision mesh filename=package://rccn_kuka_robot_cell/meshes/rail/collision/west_p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 scale=0.001 0.001 0.001; visual mesh filename=package://rccn_kuka_robot_cell/meshes/rail/visual/west_plat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
- link west_e1_rail: geometry collision mesh filename=package://rccn_kuka_robot_cell/meshes/rail/collision/west_r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 scale=0.001 0.001 0.001; visual mesh filename=package://rccn_kuka_robot_cell/meshes/rail/visual/west_rail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

File: robot_description/rccn_kuka_robot_cell/urdf/rccn_kuka_robot_cell.xacro (robot description, xacro)
@@ -12,5 +12,5 @@
             <collision>
                 <geometry>
-                    <mesh scale="0.001 0.001 0.001" filename="package://rccn_kuka_robot_cell/meshes/world/collision/robot_cell_fixture.stl"/>
+                    <mesh scale="0.001 0.001 0.001" filename="package://rccn_kuka_robot_cell/meshes/world/collision/floor.stl"/>
                 </geometry>
             </collision>
