Commit message: use no servo collision mesh

File: robot_description/rccn_kuka_robot_cell/urdf/rccn_east_robot_macro.xacro (robot description, xacro)
@@ -40,5 +40,5 @@
                 <collision>
                     <geometry>
-                        <mesh scale="0.001 0.001 0.001" filename="package://rccn_kuka_robot_cell/meshes/rail/collision/east_plate.stl"/>
+                        <mesh scale="0.001 0.001 0.001" filename="package://rccn_kuka_robot_cell/meshes/rail/collision/east_plate_no_servo.stl"/>
                     </geometry>
                 </collision>

File: robot_description/rccn_kuka_robot_cell/urdf/rccn_west_robot_macro.xacro (robot description, xacro)
@@ -40,5 +40,5 @@
                 <collision>
                     <geometry>
-                        <mesh scale="0.001 0.001 0.001" filename="package://rccn_kuka_robot_cell/meshes/rail/collision/west_plate.stl"/>
+                        <mesh scale="0.001 0.001 0.001" filename="package://rccn_kuka_robot_cell/meshes/rail/collision/west_plate_no_servo.stl"/>
                     </geometry>
                 </collision>

Commit message: add new launch

File: robot_description/rccn_kuka_robot_cell/urdf/rccn_east_robot_macro.xacro (robot description, xacro)
@@ -18,4 +18,8 @@
                     </geometry>
                 </collision>
+                <inertial>
+                    <mass value="1.0"/> <origin xyz="0 0 0" rpy="0 0 0"/>
+                    <inertia ixx="10.0" ixy="0.0" ixz="0.0" iyy="10.0" iyz="0.0" izz="10.0"/>
+                </inertial>
             </link>
             <joint name="${prefix}east_joint_e1" type="prismatic">
@@ -43,4 +47,8 @@
                     </geometry>
                 </collision>
+                <inertial>
+                    <mass value="1.0"/> <origin xyz="0 0 0" rpy="0 0 0"/>
+                    <inertia ixx="10.0" ixy="0.0" ixz="0.0" iyy="10.0" iyz="0.0" izz="10.0"/>
+                </inertial>
             </link>
             <joint name="${east_prefix}attachment_joint" type="fixed">

File: robot_description/rccn_kuka_robot_cell/urdf/rccn_kuka_robot_cell.xacro (robot description, xacro)
@@ -15,4 +15,8 @@
                 </geometry>
             </collision>
+            <inertial>
+                <mass value="100.0"/> <origin xyz="0 0 0" rpy="0 0 0"/>
+                <inertia ixx="10.0" ixy="0.0" ixz="0.0" iyy="10.0" iyz="0.0" izz="10.0"/>
+            </inertial>
         </link>
         <!--KUKA East Robot-->

File: robot_description/rccn_kuka_robot_cell/urdf/rccn_west_robot_macro.xacro (robot description, xacro)
@@ -18,4 +18,8 @@
                     </geometry>
                 </collision>
+                <inertial>
+                    <mass value="1.0"/> <origin xyz="0 0 0" rpy="0 0 0"/>
+                    <inertia ixx="10.0" ixy="0.0" ixz="0.0" iyy="10.0" iyz="0.0" izz="10.0"/>
+                </inertial>
             </link>
             <joint name="${prefix}west_joint_e1" type="prismatic">
@@ -43,4 +47,8 @@
                     </geometry>
                 </collision>
+                <inertial>
+                    <mass value="1.0"/> <origin xyz="0 0 0" rpy="0 0 0"/>
+                    <inertia ixx="10.0" ixy="0.0" ixz="0.0" iyy="10.0" iyz="0.0" izz="10.0"/>
+                </inertial>
             </link>
             <joint name="${west_prefix}attachment_joint" type="fixed">
